Commit message: Height adjustment

File: mrp2_description/urdf/base/base.urdf.xacro (robot description, xacro)
@@ -72,5 +72,5 @@
     <link name="${name}_footprint"/>
     <joint name="${name}_footprint_joint" type="fixed">
-      <origin xyz="0 0 ${wheel_radius}" rpy="0 0 0" />
+      <origin xyz="0 0 0" rpy="0 0 0" />
       <child link="${name}_link" />
       <parent link="${name}_footprint"/>

File: mrp2_description/urdf/wheels/wheel.left.urdf.xacro (robot description, xacro)
@@ -43,5 +43,5 @@
       <parent link="${parent}_link"/>
       <child link="wheel_${side}_link"/>
-      <origin xyz="0 0.2395 0.1" rpy="0 0 0"/>
+      <origin xyz="0 0.2395 ${radius}" rpy="0 0 0"/>
       <axis xyz="0 1 0"/>
       <limit effort="${torque*2}" velocity="${velocity / radius}"/>

File: mrp2_description/urdf/wheels/wheel.right.urdf.xacro (robot description, xacro)
@@ -43,5 +43,5 @@
       <parent link="${parent}_link"/>
       <child link="wheel_${side}_link"/>
-      <origin xyz="0 -0.2395 0.1" rpy="0 0 0"/>
+      <origin xyz="0 -0.2395 ${radius}" rpy="0 0 0"/>
       <axis xyz="0 1 0"/>
       <limit effort="${torque*2}" velocity="${velocity / radius}"/>

Commit message: Added sonar sensors to URDF

File: mrp2_description/urdf/base/base.urdf.xacro (robot description, xacro)
@@ -7,4 +7,5 @@
   <xacro:include filename="$(find mrp2_description)/urdf/sensors/hokuyo_utm_30lx_laser.urdf.xacro"/>
   <xacro:include filename="$(find mrp2_description)/urdf/sensors/imu.urdf.xacro"/>
+  <xacro:include filename="$(find mrp2_description)/urdf/sensors/sonar.urdf.xacro"/>
   <!-- Wheel characteristics -->
   <property name="wheel_radius"     value="0.100"/>
@@ -81,4 +82,26 @@
     <xacro:caster side="back_left" radius="${caster_radius}" width="${caster_width}" position_x="-0.213" position_y="0.141" position_z="0.0971" offset_x="-0.030" offset_y="0" offset_z="-0.0596" parent="${name}"/>
     <xacro:caster side="back_right" radius="${caster_radius}" width="${caster_width}" position_x="-0.213" position_y="-0.141" position_z="0.0971" offset_x="-0.030" offset_y="0" offset_z="-0.0596" parent="${name}"/>
+    <!-- Sonar sensors -->
+    <xacro:sonar_sensor name="${name}_sonar_1" parent="${name}" ros_topic="sonar_1" update_rate="20" maxRange="4.0" minRange="0.01" fov="${35 * deg_to_rad}" radiation="ultrasound">
+      <origin xyz="0.2688 0.17956 0.06155" rpy="0 0 ${30 * deg_to_rad}"/>
+    </xacro:sonar_sensor>
+    <xacro:sonar_sensor name="${name}_sonar_2" parent="${name}" ros_topic="sonar_2" update_rate="20" maxRange="4.0" minRange="0.01" fov="${35 * deg_to_rad}" radiation="ultrasound">
+      <origin xyz="0.28947 0.09241 0.06155" rpy="0 0 ${12 * deg_to_rad}"/>
+    </xacro:sonar_sensor>
+    <xacro:sonar_sensor name="${name}_sonar_3" parent="${name}" ros_topic="sonar_3" update_rate="20" maxRange="4.0" minRange="0.01" fov="${35 * deg_to_rad}" radiation="ultrasound">
+      <origin xyz="0.29671 0.0 0.06155" rpy="0 0 ${0 * deg_to_rad}"/>
+    </xacro:sonar_sensor>
+    <xacro:sonar_sensor name="${name}_sonar_4" parent="${name}" ros_topic="sonar_4" update_rate="20" maxRange="4.0" minRange="0.01" fov="${35 * deg_to_rad}" radiation="ultrasound">
+      <origin xyz="0.28947 -0.09241 0.06155" rpy="0 0 ${-12 * deg_to_rad}"/>
+    </xacro:sonar_sensor>
+    <xacro:sonar_sensor name="${name}_sonar_5" parent="${name}" ros_topic="sonar_5" update_rate="20" maxRange="4.0" minRange="0.01" fov="${35 * deg_to_rad}" radiation="ultrasound">
+      <origin xyz="0.2688 -0.17956 0.06155" rpy="0 0 ${-30 * deg_to_rad}"/>
+    </xacro:sonar_sensor>
+    <xacro:sonar_sensor name="${name}_sonar_6" parent="${name}" ros_topic="sonar_6" update_rate="20" maxRange="4.0" minRange="0.01" fov="${35 * deg_to_rad}" radiation="ultrasound">
+      <origin xyz="-0.25648 -0.10103 0.28155" rpy="0 0 ${180 * deg_to_rad}"/>
+    </xacro:sonar_sensor>
+    <xacro:sonar_sensor name="${name}_sonar_7" parent="${name}" ros_topic="sonar_7" update_rate="20" maxRange="4.0" minRange="0.01" fov="${35 * deg_to_rad}" radiation="ultrasound">
+      <origin xyz="-0.25648 0.10103 0.28155" rpy="0 0 ${180 * deg_to_rad}"/>
+    </xacro:sonar_sensor>
   </xacro:macro>
 </robot>

File: mrp2_description/urdf/sensors/hokuyo_utm_30lx_laser.gazebo.xacro (robot description, xacro)
@@ -6,5 +6,5 @@
         <pose>0 0 0 0 0 0</pose>
         <update_rate>${update_rate}</update_rate>
-        <visualize>true</visualize>
+        <visualize>false</visualize>
         <ray>
           <scan>

Commit message: parameterized the wheels

File: mrp2_description/urdf/base/base.urdf.xacro (robot description, xacro)
@@ -2,6 +2,7 @@
 <robot xmlns:xacro="http://ros.org/wiki/xacro">
   <xacro:include filename="$(find mrp2_description)/urdf/deg_to_rad.xacro"/>
-  <xacro:include filename="$(find mrp2_description)/urdf/wheels/wheel.right.urdf.xacro"/>
-  <xacro:include filename="$(find mrp2_description)/urdf/wheels/wheel.left.urdf.xacro"/>
+  <xacro:include filename="$(find mrp2_description)/urdf/wheels/wheel.urdf.xacro"/>
+  <!--xacro:include filename="$(find mrp2_description)/urdf/wheels/wheel.right.urdf.xacro"/>
+  <xacro:include filename="$(find mrp2_description)/urdf/wheels/wheel.left.urdf.xacro"/-->
   <xacro:include filename="$(find mrp2_description)/urdf/wheels/75mm.caster.urdf.xacro"/>
   <xacro:include filename="$(find mrp2_description)/urdf/sensors/hokuyo_utm_30lx_laser.urdf.xacro"/>
@@ -75,5 +76,5 @@
     </xacro:imu_sensor>
     <!-- Wheels -->
-    <xacro:wheel_right
+    <xacro:wheel
       side="right"
       reflect="-1.0"
@@ -82,7 +83,7 @@
       torque="${wheel_torque}"
       velocity="${wheel_velocity}"
-      separation="${wheel_separation}"
+      separation="-${wheel_separation}"
       parent="${name}"/>
-    <xacro:wheel_left
+    <xacro:wheel
       side="left"
       reflect="1.0"

File: mrp2_description/urdf/wheels/wheel.urdf.xacro (robot description, xacro)
@@ -3,5 +3,5 @@
   <xacro:include filename="$(find mrp2_description)/urdf/wheels/wheel.transmission.xacro"/>
   <xacro:include filename="$(find mrp2_description)/urdf/wheels/wheel.gazebo.xacro"/>
-  <xacro:macro name="wheel_left" params="side reflect radius width torque velocity separation parent">
+  <xacro:macro name="wheel" params="side reflect radius width torque velocity separation parent">
     <link name="wheel_${side}_link">
       <inertial>
@@ -22,5 +22,5 @@
         <origin xyz="0 0 0" rpy="0 0 0"/>
         <geometry>
-          <mesh filename="package://mrp2_description/meshes/left_wheel.stl"/>
+          <mesh filename="package://mrp2_description/meshes/${side}_wheel.stl"/>
         </geometry>
         <material name="DarkGrey"/>

Commit message: corrected imu configuration

File: mrp2_description/urdf/base/base.urdf.xacro (robot description, xacro)
@@ -74,8 +74,4 @@
     <xacro:uv_tower name="${name}_uv_tower" parent="${name}_link" >
     </xacro:uv_tower>
-    <!-- IMU -->
-    <xacro:imu_sensor name="${name}_imu" parent="${name}_link" update_rate="50.0">
-      <origin xyz="0.1604 0 0.2440" rpy="0 ${0 * deg_to_rad} ${0 * deg_to_rad}"/>
-    </xacro:imu_sensor>
     <!-- Wheels -->
     <xacro:wheel
@@ -102,4 +98,8 @@
     <xacro:caster side="back_left" radius="${caster_radius}" width="${caster_width}" position_x="-0.192" position_y="0.144" position_z="0.0971" offset_x="-0.030" offset_y="0" offset_z="-0.0596" parent="${name}"/>
     <xacro:caster side="back_right" radius="${caster_radius}" width="${caster_width}" position_x="-0.192" position_y="-0.144" position_z="0.0971" offset_x="-0.030" offset_y="0" offset_z="-0.0596" parent="${name}"/>
+    <!-- IMU -->
+    <xacro:imu_sensor name="${name}_imu" parent="${name}_link" update_rate="50.0">
+      <origin xyz="0.1604 0 0.2440" rpy="0 ${0 * deg_to_rad} ${0 * deg_to_rad}"/>
+    </xacro:imu_sensor>
     <!-- Sonar sensors -->
     <xacro:sonar_sensor name="${name}_sonar_1" parent="${name}" ros_topic="sonar_1" update_rate="20" maxRange="4.0" minRange="0.01" fov="${35 * deg_to_rad}" radiation="ultrasound">

File: mrp2_description/urdf/sensors/imu.urdf.xacro (robot description, xacro)
@@ -18,5 +18,15 @@
         <always_on>1</always_on>
         <update_rate>100.0</update_rate>
-        <imu>
+        <plugin filename="libgazebo_ros_imu_sensor.so" name="imu_plugin">
+          <topicName>imu</topicName>
+          <bodyName>base_imu_link</bodyName>
+          <updateRateHZ>10.0</updateRateHZ>
+          <gaussianNoise>0.0</gaussianNoise>
+          <xyzOffset>0 0 0</xyzOffset>
+          <rpyOffset>0 0 0</rpyOffset>
+          <frameName>base_imu_link</frameName>
+          <initialOrientationAsReference>false</initialOrientationAsReference>
+        </plugin>
+        <!--imu>
           <noise>
             <type>gaussian</type>
@@ -34,5 +44,5 @@
             </accel>
           </noise>
-        </imu>
+        </imu-->
       </sensor>
     </gazebo>
