Commit message: Organized code and structure

File: mrp2_description/gazebo/gazebo.urdf.xacro (robot description, xacro)
@@ -1,10 +1,3 @@
 <?xml version="1.0"?>
-<!--
-  Copyright (c) 2011, PAL Robotics, S.L.
-  All rights reserved.
-  This work is licensed under the Creative Commons Attribution-NonCommercial-NoDerivs 3.0 Unported License.
-  To view a copy of this license, visit http://creativecommons.org/licenses/by-nc-nd/3.0/ or send a letter to
-  Creative Commons, 444 Castro Street, Suite 900, Mountain View, California, 94041, USA.
--->
 <robot xmlns:sensor="http://playerstage.sourceforge.net/gazebo/xmlschema/#sensor"
        xmlns:controller="http://playerstage.sourceforge.net/gazebo/xmlschema/#controller"
@@ -23,5 +16,4 @@
     </plugin>
   </gazebo>
-  <!-- define global properties -->
-  <property name="M_PI" value="3.1415926535897931" />
+  <property name="M_PI" value="3.14159" />
 </robot>

File: mrp2_description/robots/mrp2_full.urdf.xacro (robot description, xacro)
@@ -1,20 +1,7 @@
 <?xml version="1.0"?>
-<!--
-  Copyright (c) 2014, PAL Robotics, S.L.
-  All rights reserved.
-  This work is licensed under the Creative Commons Attribution-NonCommercial-NoDerivs 3.0 Unported License.
-  To view a copy of this license, visit http://creativecommons.org/licenses/by-nc-nd/3.0/ or send a letter to
-  Creative Commons, 444 Castro Street, Suite 900, Mountain View, California, 94041, USA.
--->
-<robot  xmlns:xacro="http://www.ros.org/wiki/xacro"
-        name="mrp2" >
-  <!-- The following included files set up definitions of parts of the robot body -->
-  <!-- Materials for visualization -->
+<robot  xmlns:xacro="http://www.ros.org/wiki/xacro" name="mrp2" >
   <xacro:include filename="$(find mrp2_description)/urdf/materials.urdf.xacro" />
-  <!-- Base -->
   <xacro:include filename="$(find mrp2_description)/urdf/base/base.urdf.xacro" />
-    <!-- Generic simulator_gazebo plugins -->
   <xacro:include filename="$(find mrp2_description)/gazebo/gazebo.urdf.xacro" />
-  <!-- Now we can start using the macros included above to define the actual robot -->
   <xacro:base name="base"/>
 </robot>

File: mrp2_description/urdf/base/base.urdf.xacro (robot description, xacro)
@@ -1,10 +1,3 @@
 <?xml version="1.0"?>
-<!--
-  Copyright (c) 2011-2014, PAL Robotics, S.L.
-  All rights reserved.
-  This work is licensed under the Creative Commons Attribution-NonCommercial-NoDerivs 3.0 Unported License.
-  To view a copy of this license, visit http://creativecommons.org/licenses/by-nc-nd/3.0/ or send a letter to
-  Creative Commons, 444 Castro Street, Suite 900, Mountain View, California, 94041, USA.
--->
 <robot xmlns:xacro="http://ros.org/wiki/xacro">
   <xacro:include filename="$(find mrp2_description)/urdf/deg_to_rad.xacro"/>
@@ -12,9 +5,6 @@
   <xacro:include filename="$(find mrp2_description)/urdf/wheels/wheel.left.urdf.xacro"/>
   <xacro:include filename="$(find mrp2_description)/urdf/wheels/75mm.caster.urdf.xacro"/>
-  <xacro:include filename="$(find mrp2_description)/urdf/sensors/range.urdf.xacro"/>
   <xacro:include filename="$(find mrp2_description)/urdf/sensors/hokuyo_utm_30lx_laser.urdf.xacro"/>
   <xacro:include filename="$(find mrp2_description)/urdf/sensors/imu.urdf.xacro"/>
-  <xacro:include filename="$(find mrp2_description)/urdf/objects/cover.urdf.xacro"/>
-  <xacro:include filename="$(find mrp2_description)/urdf/objects/antenna.urdf.xacro"/>
   <!-- Wheel characteristics -->
   <property name="wheel_radius"     value="0.102"/>
@@ -76,54 +66,4 @@
       <parent link="${name}_footprint"/>
     </joint>
-    <!-- ADROBOT ADDITION -->
-    <!--
-    <link name="${name}_adrobot_link">
-      <inertial>
-      <origin
-        xyz="0.0 0.0 0.0"
-        rpy="0 0 0" />
-      <mass
-        value="3.75049" />
-      <inertia
-        ixx="1.40843"
-        ixy="-0.00047"
-        ixz="-0.01284"
-        iyy="1.69950"
-        iyz="0.00099"
-        izz="1.30459" />
-    </inertial>
-      <visual>
-        <origin xyz="0 0 0" rpy="0 0 0" />
-        <geometry>
-          <mesh filename="package://mrp2_description/meshes/adrobot_s.stl" />
-        </geometry>
-        <material name="SkyBlue" />
-      </visual>
-      <collision>
-        <origin xyz="0 0 0" rpy="0 0 0" />
-        <geometry>
-          <mesh filename="package://mrp2_description/meshes/adrobot_s.stl" />
-        </geometry>
-      </collision>
-    </link>
-    <gazebo reference="${name}_adrobot_link">
-      <material>Gazebo/White</material>
-    </gazebo>
-    <joint name="${name}_adrobot_joint" type="fixed">
-      <origin xyz="-0.4 -0.372 0.3" rpy="${0 * deg_to_rad} 0 0" />
-      <child link="${name}_adrobot_link" />
-      <parent link="${name}_link"/>
-    </joint>
-	-->
-    <!-- ADROBOT ADDITION -->
-    <!-- Orange cover & antennas -->
-    <!--<xacro:antenna name="${name}_antenna_left" parent="${name}_link">
-      <origin xyz="-0.201 0.1062 0.195" rpy="0 0 0"/>
-    </xacro:antenna>
-    <xacro:antenna name="${name}_antenna_right" parent="${name}_link">
-      <origin xyz="-0.201 -0.1062 0.195" rpy="0 0 0"/>
-    </xacro:antenna>-->
-    <!-- Laser -->
-    <!-- Theoretic FOV = 220 -->
     <xacro:hokuyo_utm_30lx_laser name="${name}_laser" parent="${name}" ros_topic="scan" update_rate="10" min_angle="${-135 * deg_to_rad}" max_angle="${135 * deg_to_rad}" >
       <origin xyz="${base_laser_x} ${base_laser_y} ${base_laser_z}" rpy="0 0 0" />
@@ -133,15 +73,4 @@
       <origin xyz="0.200 0 0.200" rpy="0 ${0 * deg_to_rad} ${0 * deg_to_rad}"/>
     </xacro:imu_sensor>
-    <!-- Sonars -->
-    <!--<xacro:range_sensor name="${name}_sonar_1" parent="${name}" ros_topic="sonar_${name}" update_rate="5" maxRange="0.75" minRange="0.01" fov="0.5" radiation="ultrasound">
-      <origin xyz="-0.183 0.183 0.173" rpy="0 0 ${135 * deg_to_rad}"/>
-    </xacro:range_sensor>
-    <xacro:range_sensor name="${name}_sonar_2" parent="${name}" ros_topic="sonar_${name}" update_rate="5" maxRange="0.75" minRange="0.01" fov="0.5" radiation="ultrasound">
-      <origin xyz="-0.259 0.0 0.173" rpy="0 0 ${180 * deg_to_rad}"/>
-    </xacro:range_sensor>
-    <xacro:range_sensor name="${name}_sonar_3" parent="${name}" ros_topic="sonar_${name}" update_rate="5" maxRange="0.75" minRange="0.01" fov="0.5" radiation="ultrasound">
-      <origin xyz="-0.183 -0.183 0.173" rpy="0 0 ${225 * deg_to_rad}"/>
-    </xacro:range_sensor>
-    -->
     <!-- Wheels -->
     <xacro:wheel_right side="right" reflect="-1.0" radius="${wheel_radius}" width="${wheel_width}" torque="${wheel_torque}" velocity="${wheel_velocity}" separation="${wheel_separation}" parent="${name}"/>

File: mrp2_description/urdf/materials.urdf.xacro (robot description, xacro)
@@ -1,10 +1,3 @@
 <?xml version="1.0"?>
-<!--
-  Copyright (c) 2011, PAL Robotics, S.L.
-  All rights reserved.
-  This work is licensed under the Creative Commons Attribution-NonCommercial-NoDerivs 3.0 Unported License.
-  To view a copy of this license, visit http://creativecommons.org/licenses/by-nc-nd/3.0/ or send a letter to
-  Creative Commons, 444 Castro Street, Suite 900, Mountain View, California, 94041, USA.
--->
 <robot>
   <material name="Blue">

File: mrp2_description/urdf/sensors/hokuyo_urg_04lx_ug01_laser.gazebo.xacro (robot description, xacro)
@@ -1,12 +1,3 @@
 <?xml version="1.0"?>
-<!--
-  Copyright (c) 2011, PAL Robotics, S.L.
-  All rights reserved.
-  This work is licensed under the Creative Commons Attribution-NonCommercial-NoDerivs 3.0 Unported License.
-  To view a copy of this license, visit http://creativecommons.org/licenses/by-nc-nd/3.0/ or send a letter to
-  Creative Commons, 444 Castro Street, Suite 900, Mountain View, California, 94041, USA.
-  Laser configuration according with the Hokuyo URG-04LX-UG01 product specification:
-  http://www.hokuyo-aut.jp/02sensor/07scanner/download/products/urg-04lx-ug01/data/URG-04LX_UG01_spec_en.pdf
--->
 <robot xmlns:xacro="http://ros.org/wiki/xacro">
   <xacro:macro name="hokuyo_urg_04lx_ug01_laser_gazebo" params="name ros_topic update_rate min_angle max_angle">
@@ -19,7 +10,6 @@
           <scan>
             <horizontal>
-              <!-- 683 steps in 240deg fov -->
               <samples>${683*(max_angle - min_angle)/(240.0 * deg_to_rad)}</samples>
-              <resolution>1</resolution> <!-- not the sensor resolution; just 1 -->
+              <resolution>1</resolution>
               <min_angle>${min_angle}</min_angle>
               <max_angle>${max_angle}</max_angle>

File: mrp2_description/urdf/sensors/hokuyo_urg_04lx_ug01_laser.urdf.xacro (robot description, xacro)
@@ -1,10 +1,3 @@
 <?xml version="1.0"?>
-<!--
-  Copyright (c) 2011, PAL Robotics, S.L.
-  All rights reserved.
-  This work is licensed under the Creative Commons Attribution-NonCommercial-NoDerivs 3.0 Unported License.
-  To view a copy of this license, visit http://creativecommons.org/licenses/by-nc-nd/3.0/ or send a letter to
-  Creative Commons, 444 Castro Street, Suite 900, Mountain View, California, 94041, USA.
--->
 <robot xmlns:xacro="http://ros.org/wiki/xacro">
   <xacro:include filename="$(find mrp2_description)/urdf/sensors/hokuyo_urg_04lx_ug01_laser.gazebo.xacro" />
@@ -32,5 +25,4 @@
       <child  link="${name}_link"/>
     </joint>
-    <!-- gazebo extensions -->
     <xacro:hokuyo_urg_04lx_ug01_laser_gazebo name="${name}" ros_topic="${ros_topic}" update_rate="${update_rate}" min_angle="${min_angle}" max_angle="${max_angle}" />
   </xacro:macro>

File: mrp2_description/urdf/sensors/hokuyo_utm_30lx_laser.gazebo.xacro (robot description, xacro)
@@ -1,12 +1,3 @@
 <?xml version="1.0"?>
-<!--
-  Copyright (c) 2011, PAL Robotics, S.L.
-  All rights reserved.
-  This work is licensed under the Creative Commons Attribution-NonCommercial-NoDerivs 3.0 Unported License.
-  To view a copy of this license, visit http://creativecommons.org/licenses/by-nc-nd/3.0/ or send a letter to
-  Creative Commons, 444 Castro Street, Suite 900, Mountain View, California, 94041, USA.
-  Laser configuration according with the Hokuyo URG-04LX-UG01 product specification:
-  http://www.hokuyo-aut.jp/02sensor/07scanner/download/products/urg-04lx-ug01/data/URG-04LX_UG01_spec_en.pdf
--->
 <robot xmlns:xacro="http://ros.org/wiki/xacro">
   <xacro:macro name="hokuyo_utm_30lx_laser_gazebo" params="name ros_topic update_rate min_angle max_angle">
@@ -19,7 +10,6 @@
           <scan>
             <horizontal>
-              <!-- 683 steps in 240deg fov -->
-              <samples>${683*(max_angle - min_angle)/(240.0 * deg_to_rad)}</samples>
-              <resolution>1</resolution> <!-- not the sensor resolution; just 1 -->
+              <samples>${1080.0*(max_angle - min_angle)/(270.0 * deg_to_rad)}</samples>
+              <resolution>1</resolution>
               <min_angle>${min_angle}</min_angle>
               <max_angle>${max_angle}</max_angle>

File: mrp2_description/urdf/sensors/hokuyo_utm_30lx_laser.urdf.xacro (robot description, xacro)
@@ -1,10 +1,3 @@
 <?xml version="1.0"?>
-<!--
-  Copyright (c) 2011, PAL Robotics, S.L.
-  All rights reserved.
-  This work is licensed under the Creative Commons Attribution-NonCommercial-NoDerivs 3.0 Unported License.
-  To view a copy of this license, visit http://creativecommons.org/licenses/by-nc-nd/3.0/ or send a letter to
-  Creative Commons, 444 Castro Street, Suite 900, Mountain View, California, 94041, USA.
--->
 <robot xmlns:xacro="http://ros.org/wiki/xacro">
   <xacro:include filename="$(find mrp2_description)/urdf/sensors/hokuyo_utm_30lx_laser.gazebo.xacro" />
@@ -32,5 +25,4 @@
       <child  link="${name}_link"/>
     </joint>
-    <!-- gazebo extensions -->
     <xacro:hokuyo_utm_30lx_laser_gazebo name="${name}" ros_topic="${ros_topic}" update_rate="${update_rate}" min_angle="${min_angle}" max_angle="${max_angle}" />
   </xacro:macro>

File: mrp2_description/urdf/sensors/imu.urdf.xacro (robot description, xacro)
@@ -1,10 +1,3 @@
 <?xml version="1.0"?>
-<!--
-  Copyright (c) 2011-2012, PAL Robotics, S.L.
-  All rights reserved.
-  This work is licensed under the Creative Commons Attribution-NonCommercial-NoDerivs 3.0 Unported License.
-  To view a copy of this license, visit http://creativecommons.org/licenses/by-nc-nd/3.0/ or send a letter to
-  Creative Commons, 444 Castro Street, Suite 900, Mountain View, California, 94041, USA.
--->
 <robot xmlns:xacro="http://ros.org/wiki/xacro">
   <xacro:macro name="imu_sensor" params="name parent *origin update_rate">
@@ -15,10 +8,4 @@
         <inertia ixx="0.000001" ixy="0" ixz="0" iyy="0.000001" iyz="0" izz="0.000001"/>
       </inertial>
-      <!--visual>
-        <origin rpy="0 0 0" xyz="0 0 0"/>
-        <geometry>
-          <box size="0.01 0.01 0.01"/>
-        </geometry>
-      </visual-->
     </link>
     <joint name="${name}_joint" type="fixed">

File: mrp2_description/urdf/wheels/75mm.caster.urdf.xacro (robot description, xacro)
@@ -1,10 +1,3 @@
 <?xml version="1.0"?>
-<!--
-  Copyright (c) 2014, PAL Robotics, S.L.
-  All rights reserved.
-  This work is licensed under the Creative Commons Attribution-NonCommercial-NoDerivs 3.0 Unported License.
-  To view a copy of this license, visit http://creativecommons.org/licenses/by-nc-nd/3.0/ or send a letter to
-  Creative Commons, 444 Castro Street, Suite 900, Mountain View, California, 94041, USA.
--->
 <robot xmlns:xacro="http://ros.org/wiki/xacro">
   <xacro:include filename="$(find mrp2_description)/urdf/wheels/caster.transmission.xacro"/>
@@ -61,8 +54,4 @@
       <axis xyz="0 1 0"/>
     </joint>
-    <!-- Transmission 132.1 mm-->
-    <!--xacro:caster_transmission name="" side="${side}" number="" reduction=""-->
-    <!-- Gazebo extensions -->
-    <!--<xacro:caster_gazebo side="${side}"/>-->
     <xacro:caster_gazebo side="${side}"/>
   </xacro:macro>

File: mrp2_description/urdf/wheels/caster.gazebo.xacro (robot description, xacro)
@@ -1,13 +1,5 @@
 <?xml version="1.0"?>
-<!--
-  Copyright (c) 2011, PAL Robotics, S.L.
-  All rights reserved.
-  This work is licensed under the Creative Commons Attribution-NonCommercial-NoDerivs 3.0 Unported License.
-  To view a copy of this license, visit http://creativecommons.org/licenses/by-nc-nd/3.0/ or send a letter to
-  Creative Commons, 444 Castro Street, Suite 900, Mountain View, California, 94041, USA.
--->
 <robot xmlns:xacro="http://ros.org/wiki/xacro">
   <xacro:macro name="caster_gazebo" params="side">
-    <!-- Contact model for the caster wheel surface -->
     <gazebo reference="caster_${side}_2_link">
       <kp>1000000.0</kp>

File: mrp2_description/urdf/wheels/caster.transmission.xacro (robot description, xacro)
@@ -1,12 +1,4 @@
 <?xml version="1.0"?>
-<!--
-  Copyright (c) 2011-2014, PAL Robotics, S.L.
-  All rights reserved.
-  This work is licensed under the Creative Commons Attribution-NonCommercial-NoDerivs 3.0 Unported License.
-  To view a copy of this license, visit http://creativecommons.org/licenses/by-nc-nd/3.0/ or send a letter to
-  Creative Commons, 444 Castro Street, Suite 900, Mountain View, California, 94041, USA.
--->
 <robot xmlns:xacro="http://ros.org/wiki/xacro">
-  <!-- Caster transmissions -->
   <xacro:macro name="caster_transmission" params="name side number reduction" >
     <transmission name="${name}_${side}_${number}_trans">

File: mrp2_description/urdf/wheels/wheel.gazebo.xacro (robot description, xacro)
@@ -1,13 +1,5 @@
 <?xml version="1.0"?>
-<!--
-  Copyright (c) 2011, PAL Robotics, S.L.
-  All rights reserved.
-  This work is licensed under the Creative Commons Attribution-NonCommercial-NoDerivs 3.0 Unported License.
-  To view a copy of this license, visit http://creativecommons.org/licenses/by-nc-nd/3.0/ or send a letter to
-  Creative Commons, 444 Castro Street, Suite 900, Mountain View, California, 94041, USA.
--->
 <robot xmlns:xacro="http://ros.org/wiki/xacro">
   <xacro:macro name="wheel_gazebo" params="side">
-    <!-- Contact model for the wheel surface -->
     <gazebo reference="wheel_${side}_link">
       <mu1 value="1.0"/>

File: mrp2_description/urdf/wheels/wheel.left.urdf.xacro (robot description, xacro)
@@ -1,10 +1,3 @@
 <?xml version="1.0"?>
-<!--
-  Copyright (c) 2014, PAL Robotics, S.L.
-  All rights reserved.
-  This work is licensed under the Creative Commons Attribution-NonCommercial-NoDerivs 3.0 Unported License.
-  To view a copy of this license, visit http://creativecommons.org/licenses/by-nc-nd/3.0/ or send a letter to
-  Creative Commons, 444 Castro Street, Suite 900, Mountain View, California, 94041, USA.
--->
 <robot xmlns:xacro="http://ros.org/wiki/xacro">
   <xacro:include filename="$(find mrp2_description)/urdf/wheels/wheel.transmission.xacro"/>
@@ -47,20 +40,7 @@
       <limit effort="${torque*2}" velocity="${velocity / radius}"/>
     </joint>
-    <!--<gazebo reference="wheel_${side}_link">
-      <velocity_decay>
-        <linear>0.2</linear>
-        <angular>0.4</angular>
-      </velocity_decay>
-    </gazebo>
-    <gazebo reference="wheel_${side}_link">
-      <mu1>0.2</mu1>
-      <mu2>0.2</mu2>
-    </gazebo>-->
     <gazebo reference="wheel_${side}_link">
       <material>Gazebo/DarkGrey</material>
     </gazebo>
-        <!-- Transmission -->
-    <!--<xacro:wheel_transmission side="${side}"/>-->
-    <!-- Gazebo extensions -->
     <xacro:wheel_gazebo side="${side}"/>
   </xacro:macro>

File: mrp2_description/urdf/wheels/wheel.right.urdf.xacro (robot description, xacro)
@@ -1,10 +1,3 @@
 <?xml version="1.0"?>
-<!--
-  Copyright (c) 2014, PAL Robotics, S.L.
-  All rights reserved.
-  This work is licensed under the Creative Commons Attribution-NonCommercial-NoDerivs 3.0 Unported License.
-  To view a copy of this license, visit http://creativecommons.org/licenses/by-nc-nd/3.0/ or send a letter to
-  Creative Commons, 444 Castro Street, Suite 900, Mountain View, California, 94041, USA.
--->
 <robot xmlns:xacro="http://ros.org/wiki/xacro">
   <xacro:include filename="$(find mrp2_description)/urdf/wheels/wheel.transmission.xacro"/>
@@ -47,20 +40,7 @@
       <limit effort="${torque*2}" velocity="${velocity / radius}"/>
     </joint>
-    <!--<gazebo reference="wheel_${side}_link">
-      <velocity_decay>
-        <linear>0.2</linear>
-        <angular>0.4</angular>
-      </velocity_decay>
-    </gazebo>
-    <gazebo reference="wheel_${side}_link">
-      <mu1>0.2</mu1>
-      <mu2>0.2</mu2>
-    </gazebo>-->
     <gazebo reference="wheel_${side}_link">
       <material>Gazebo/DarkGrey</material>
     </gazebo>
-        <!-- Transmission -->
-    <!--<xacro:wheel_transmission side="${side}"/>-->
-    <!-- Gazebo extensions -->
     <xacro:wheel_gazebo side="${side}"/>
   </xacro:macro>

File: mrp2_description/urdf/wheels/wheel.transmission.xacro (robot description, xacro)
@@ -1,12 +1,4 @@
 <?xml version="1.0"?>
-<!--
-  Copyright (c) 2011-2014, PAL Robotics, S.L.
-  All rights reserved.
-  This work is licensed under the Creative Commons Attribution-NonCommercial-NoDerivs 3.0 Unported License.
-  To view a copy of this license, visit http://creativecommons.org/licenses/by-nc-nd/3.0/ or send a letter to
-  Creative Commons, 444 Castro Street, Suite 900, Mountain View, California, 94041, USA.
--->
 <robot xmlns:xacro="http://ros.org/wiki/xacro">
-  <!-- Wheel transmission -->
   <xacro:macro name="wheel_transmission" params="side">
     <transmission name="wheel_${side}_trans">
