Commit message: initial commit: switch from custom plugin to gazebo diff drive

File: mrp2_description/gazebo/gazebo.urdf.xacro (robot description, xacro)
@@ -1,10 +1,11 @@
 <?xml version="1.0"?>
-<robot xmlns:sensor="http://playerstage.sourceforge.net/gazebo/xmlschema/#sensor"
+<robot xmlns:xacro="http://www.ros.org/wiki/xacro"
+       xmlns:sensor="http://playerstage.sourceforge.net/gazebo/xmlschema/#sensor"
        xmlns:controller="http://playerstage.sourceforge.net/gazebo/xmlschema/#controller"
        xmlns:interface="http://playerstage.sourceforge.net/gazebo/xmlschema/#interface">
   <gazebo>
     <plugin filename="libgazebo_ros_control.so" name="ros_control">
-      <ns></ns>
-      <robotSimType>mrp2_hardware_gazebo/Mrp2HardwareGazebo</robotSimType>
+      <!-- <robotNamespace></robotNamespace>
+           <robotSimType>mrp2_hardware_gazebo/Mrp2HardwareGazebo</robotSimType> -->
       <controlPeriod>0.001</controlPeriod>
     </plugin>
@@ -15,5 +16,23 @@
       <updateRate>100.0</updateRate>
     </plugin>
+    <plugin filename="libgazebo_ros_diff_drive.so" name="differential_drive_controller">
+      <updateRate>180</updateRate>
+      <leftJoint>wheel_left_joint</leftJoint>
+      <rightJoint>wheel_right_joint</rightJoint>
+      <wheelSeparation>0.5380</wheelSeparation>
+      <wheelDiameter>0.2410</wheelDiameter>
+      <wheelAcceleration>1.0</wheelAcceleration>
+      <wheelTorque>20</wheelTorque>
+      <commandTopic>cmd_vel</commandTopic>
+      <odometryTopic>odom</odometryTopic>
+      <odometryFrame>odom</odometryFrame>
+      <robotBaseFrame>base_footprint</robotBaseFrame>
+      <odometrySource>1</odometrySource>
+      <publishWheelTF>true</publishWheelTF>
+      <publishOdom>true</publishOdom>
+      <publishWheelJointState>true</publishWheelJointState>
+      <legacyMode>false</legacyMode>
+    </plugin>
   </gazebo>
-  <property name="M_PI" value="3.14159" />
+  <xacro:property name="M_PI" value="3.14159" />
 </robot>

File: mrp2_description/urdf/base/base.urdf.xacro (robot description, xacro)
@@ -9,21 +9,21 @@
   <xacro:include filename="$(find mrp2_description)/urdf/sensors/sonar.urdf.xacro"/>
   <!-- Wheel characteristics -->
-  <property name="wheel_radius"     value="0.100"/>
-  <property name="wheel_width"      value="0.050"/>
-  <property name="wheel_separation" value="0.4715"/>
-  <property name="wheel_torque"     value="5.0"/>
-  <property name="wheel_velocity"   value="2.0"/>
+  <xacro:property name="wheel_radius"     value="0.100"/>
+  <xacro:property name="wheel_width"      value="0.050"/>
+  <xacro:property name="wheel_separation" value="0.4715"/>
+  <xacro:property name="wheel_torque"     value="5.0"/>
+  <xacro:property name="wheel_velocity"   value="2.0"/>
   <!-- Caster wheel characteristics -->
-  <property name="caster_radius"       value="0.0375"/>
-  <property name="caster_width"        value="0.020"/>
-  <property name="caster_separation_x" value="0.384"/>
-  <property name="caster_separation_y" value="0.288"/>
-  <property name="caster_offset_x"     value="-0.002"/>
-  <property name="caster_offset_y"     value="0.0"/>
-  <property name="caster_offset_z"     value="0.075"/>
+  <xacro:property name="caster_radius"       value="0.0375"/>
+  <xacro:property name="caster_width"        value="0.020"/>
+  <xacro:property name="caster_separation_x" value="0.384"/>
+  <xacro:property name="caster_separation_y" value="0.288"/>
+  <xacro:property name="caster_offset_x"     value="-0.002"/>
+  <xacro:property name="caster_offset_y"     value="0.0"/>
+  <xacro:property name="caster_offset_z"     value="0.075"/>
   <!-- Laser characteristics -->
-  <property name="base_laser_x" value="0.239"/>
-  <property name="base_laser_y" value="0.0"/>
-  <property name="base_laser_z" value="0.2660"/>
+  <xacro:property name="base_laser_x" value="0.239"/>
+  <xacro:property name="base_laser_y" value="0.0"/>
+  <xacro:property name="base_laser_z" value="0.2660"/>
   <xacro:macro name="base" params="name">
     <!-- Base -->
@@ -75,6 +75,22 @@
     </xacro:imu_sensor>
     <!-- Wheels -->
-    <xacro:wheel_right side="right" reflect="-1.0" radius="${wheel_radius}" width="${wheel_width}" torque="${wheel_torque}" velocity="${wheel_velocity}" separation="${wheel_separation}" parent="${name}"/>
-    <xacro:wheel_left side="left"  reflect="1.0" radius="${wheel_radius}" width="${wheel_width}" torque="${wheel_torque}" velocity="${wheel_velocity}" separation="${wheel_separation}" parent="${name}"/>
+    <xacro:wheel_right
+      side="right"
+      reflect="-1.0"
+      radius="${wheel_radius}"
+      width="${wheel_width}"
+      torque="${wheel_torque}"
+      velocity="${wheel_velocity}"
+      separation="${wheel_separation}"
+      parent="${name}"/>
+    <xacro:wheel_left
+      side="left"
+      reflect="1.0"
+      radius="${wheel_radius}"
+      width="${wheel_width}"
+      torque="${wheel_torque}"
+      velocity="${wheel_velocity}"
+      separation="${wheel_separation}"
+      parent="${name}"/>
     <!-- Casters wheels -->
     <xacro:caster side="front_left" radius="${caster_radius}" width="${caster_width}" position_x="0.192" position_y="0.144" position_z="0.0971" offset_x="-0.030" offset_y="0" offset_z="-0.0596" parent="${name}"/>

File: mrp2_description/urdf/sensors/imu.urdf.xacro (robot description, xacro)
@@ -12,5 +12,5 @@
       <parent link="${parent}"/>
       <child link="${name}_link"/>
-      <insert_block name="origin"/>
+      <xacro:insert_block name="origin"/>
     </joint>
     <gazebo reference="${name}_link">

Commit message: fix transforms

File: mrp2_description/gazebo/gazebo.urdf.xacro (robot description, xacro)
@@ -5,10 +5,10 @@
        xmlns:interface="http://playerstage.sourceforge.net/gazebo/xmlschema/#interface">
   <gazebo>
-    <!--plugin filename="libgazebo_ros_p3d.so" name="gazebo_ros_p3d">
+    <plugin filename="libgazebo_ros_p3d.so" name="gazebo_ros_p3d">
       <bodyName>base_footprint</bodyName>
       <topicName>ground_truth_odom</topicName>
       <alwaysOn>true</alwaysOn>
       <updateRate>20</updateRate>
-    </plugin-->
+    </plugin>
     <plugin filename="libgazebo_ros_diff_drive.so" name="differential_drive_controller">
       <updateRate>20</updateRate>
@@ -22,7 +22,7 @@
       <odometryTopic>odom</odometryTopic>
       <odometryFrame>odom</odometryFrame>
-      <robotBaseFrame>base_link</robotBaseFrame>
+      <robotBaseFrame>base_footprint</robotBaseFrame>
       <odometrySource>encoder</odometrySource>
-      <publishWheelTF>true</publishWheelTF>
+      <publishWheelTF>false</publishWheelTF>
       <publishOdom>true</publishOdom>
       <publishWheelJointState>true</publishWheelJointState>

File: mrp2_description/urdf/base/base.urdf.xacro (robot description, xacro)
@@ -4,6 +4,4 @@
   <xacro:include filename="$(find mrp2_description)/urdf/attachment/uv_tower.urdf.xacro"/>
   <xacro:include filename="$(find mrp2_description)/urdf/wheels/wheel.urdf.xacro"/>
-  <!--xacro:include filename="$(find mrp2_description)/urdf/wheels/wheel.right.urdf.xacro"/>
-  <xacro:include filename="$(find mrp2_description)/urdf/wheels/wheel.left.urdf.xacro"/-->
   <xacro:include filename="$(find mrp2_description)/urdf/wheels/75mm.caster.urdf.xacro"/>
   <xacro:include filename="$(find mrp2_description)/urdf/sensors/hokuyo_utm_30lx_laser.urdf.xacro"/>
@@ -83,5 +81,5 @@
       velocity="${wheel_velocity}"
       separation="-${wheel_separation}"
-      parent="${name}"/>
+      parent="${name}_link"/>
     <xacro:wheel
       side="left"
@@ -92,5 +90,5 @@
       velocity="${wheel_velocity}"
       separation="${wheel_separation}"
-      parent="${name}"/>
+      parent="${name}_link"/>
     <!-- Casters wheels -->
     <xacro:caster side="front_left" radius="${caster_radius}" width="${caster_width}" position_x="0.192" position_y="0.144" position_z="0.0971" offset_x="-0.030" offset_y="0" offset_z="-0.0596" parent="${name}"/>

File: mrp2_description/urdf/wheels/wheel.urdf.xacro (robot description, xacro)
@@ -34,5 +34,5 @@
     </link>
     <joint name="wheel_${side}_joint" type="continuous">
-      <parent link="${parent}_link"/>
+      <parent link="${parent}"/>
       <child link="wheel_${side}_link"/>
       <origin xyz="0 ${separation / 2} ${radius}" rpy="0 0 0"/>
